File: spoofer.kicad_sch (KiCad schematic)
At the start: 6 parts, among them J1 HDMI_A, J2 Conn_01x02, J3 HDMI_A, J4 Conn_01x03, J5 Conn_01x03, U1 AT24CS02-SSHM

Commit message: Redesign board
Now it is smaller.
Parts:
- U1: LCSC# (none) -> C6205
Changed lines of the file:
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@@
+      (effects (font (size 1.27 1.27)) hide)
+    )
+    (property "LCSC#" "C6205" (at 133.35 121.92 0)
       (effects (font (size 1.27 1.27)) hide)
     )
